Commit message: upto - firmware for arduino

File: custom_robot_sim/src/rosbots_description/urdf/rosbots.gazebo.xacro (robot description, xacro)
@@ -65,3 +65,36 @@
         </plugin>
     </gazebo>
+    <gazebo reference="wheel_left_link">
+        <mu1>1.0</mu1>
+        <mu2>1.0</mu2>
+        <kp>1000000.0</kp>
+        <kd>100.0</kd>
+        <minDepth>0.001</minDepth>
+        <maxVel>1.0</maxVel>
+        </gazebo>
+        <gazebo reference="wheel_right_link">
+        <mu1>1.0</mu1>
+        <mu2>1.0</mu2>
+        <kp>1000000.0</kp>
+        <kd>100.0</kd>
+        <minDepth>0.001</minDepth>
+        <maxVel>1.0</maxVel>
+    </gazebo>
+    <gazebo reference="base_link">
+        <material>Gazebo/Blue</material>
+        <mu1>0.3</mu1>
+        <mu2>0.3</mu2>
+        <sensor type="contact" name="bumpers">
+            <always_on>1</always_on>
+            <update_rate>50.0</update_rate>
+            <visualize>true</visualize>
+            <contact>
+            <collision>base_footprint_collision_base_link</collision>
+            </contact>
+        </sensor>
+    </gazebo>
+    <gazebo reference="camera_link">
+        <mu1>0.2</mu1>
+        <mu2>0.2</mu2>
+    </gazebo>
 </robot>

File: custom_robot_sim/src/rosbots_description/urdf/rosbots.xacro (robot description, xacro)
@@ -2,10 +2,10 @@
 <robot name="rosbots" xmlns:xacro="http://www.ros.org/wiki/xacro">
     <xacro:include filename="$(find rosbots_description)/urdf/rosbots.gazebo.xacro" />
-    <link name="base_footprint"/>
+    <!-- <link name="base_footprint"/>
     <joint name="base_joint" type="fixed">
       <origin xyz="0 0 0.05" rpy="0 0 0" />
       <parent link="base_footprint"/>
       <child link="base_link" />
-    </joint>
+    </joint> -->
     <link name="base_link">
       <visual>
